File: PERRI_the_PCB_Rev2_070822.kicad_pcb (KiCad board)
At the start: 2 copper layers, 163 x 100 mm, 42 parts, among them J1 SS5-80-3.00-X-D-K-XX, J2 Conn_01x02, J3 Conn_02x50_Counter_Clockwise, J4 Conn_02x05_Counter_Clockwise, J5 SS5-80-3.00-X-D-K-XX, J6 Conn_01x03, J7 Conn_01x03, J8 Conn_01x03, SW2 SW_DIP_x08, U1 TMP441AIDCNR, U2 TPS2595, U3 PCA9554ADB, U4 NCV8508

Commit message: made changes to rev 2
Parts:
- moved D1 7.99 mm to (234.5, 107.6)
- moved C7 7.54 mm to (138.2, 116.5), turned to 90 degrees
- moved R5 6.17 mm to (135.4, 101.9), turned to 180 degrees
- moved R15 5.56 mm to (137.6, 123.8), turned to 180 degrees
- moved R4 5.32 mm to (125.2, 69.5), turned to 90 degrees
- moved C3 3.63 mm to (224.8, 67.4), turned to 90 degrees
- moved R3 3.45 mm to (128.0, 69.6), turned to 90 degrees
- moved C4 2.96 mm to (221.0, 67.4), turned to 90 degrees
- moved C6 1.72 mm to (130.9, 69.6)
- moved C5 1.34 mm to (228.7, 112.7)
Connections:
- J1 pad 01: unconnected-(J1-Pad01) -> /12V_To_Hat
- J1 pad 03: unconnected-(J1-Pad03) -> /12V_To_Hat
- J1 pad 04: unconnected-(J1-Pad04) -> /12V_To_Hat
- J1 pad 05: unconnected-(J1-Pad05) -> /12V_To_Hat
- J1 pad 06: unconnected-(J1-Pad06) -> /12V_To_Hat
- J1 pad 07: unconnected-(J1-Pad07) -> /12V_To_Hat
- J1 pad 16: unconnected-(J1-Pad16) -> GND
- J1 pad 22: unconnected-(J1-Pad22) -> GND
- J1 pad 28: unconnected-(J1-Pad28) -> GND
- J1 pad 34: unconnected-(J1-Pad34) -> GND
- J1 pad 40: unconnected-(J1-Pad40) -> GND
- J1 pad 46: unconnected-(J1-Pad46) -> GND
- J5 pad 15: unconnected-(J5-Pad15) -> GND
- J5 pad 23: unconnected-(J5-Pad23) -> GND
- J5 pad 31: unconnected-(J5-Pad31) -> GND
- J5 pad 39: unconnected-(J5-Pad39) -> GND
- J5 pad 47: unconnected-(J5-Pad47) -> GND
- J5 pad 55: unconnected-(J5-Pad55) -> GND
- J5 pad 63: unconnected-(J5-Pad63) -> GND
Routing:
- net /To_Efuse_EN: track 0.00 -> 108.5 mm, vias 0 -> 1
- net GND: track 212.4 -> 258.2 mm, vias 23 -> 25
- net /SDA: track 297.7 -> 289.1 mm, vias 2 -> 0
- net /12V_To_Hat: track 8.64 -> 4.57 mm
- net +5V: track 0.00 -> 2.63 mm
- net Net-(C5-Pad2): track 10.2 -> 12.8 mm
- net /SCL: track 249.7 -> 252.0 mm, vias 6 -> 4
- net +12V: track 0.01 -> 1.07 mm
- net /DS_EN: vias 2 -> 0
